Commit message: fix urdf to solve stereo image not correct distance pointcloud

File: robot/robot_description/urdf/robot_thesis.gazebo.xacro (robot description, xacro)
@@ -130,5 +130,5 @@
       <visualize>$(arg camera_visual)</visualize>
       <camera>
-          <horizontal_fov>1.085595</horizontal_fov>
+          <horizontal_fov>${60.0*3.14/180.0}</horizontal_fov>
           <image>
               <width>640</width>
@@ -162,5 +162,5 @@
       <visualize>$(arg camera_visual)</visualize>
       <camera>
-          <horizontal_fov>1.085595</horizontal_fov>
+          <horizontal_fov>${60.0*3.14/180.0}</horizontal_fov>
           <image>
               <width>640</width>

File: robot/robot_description/urdf/robot_thesis.urdf.xacro (robot description, xacro)
@@ -166,5 +166,5 @@
   </link>
   <joint name="camera_left_joint" type="fixed">
-    <origin xyz="0.1 0.02 0.12" rpy="0 0 0"/>
+    <origin xyz="0.1 0.015 0.12" rpy="0 0 0"/>
     <parent link="base_link"/>
     <child link="camera_left_link"/>
@@ -191,5 +191,5 @@
   <link name="camera_left_rgb_optical_frame"/>
   <joint name="camera_right_joint" type="fixed">
-    <origin xyz="0.1 -0.02 0.12" rpy="0 0 0"/>
+    <origin xyz="0.1 -0.015 0.12" rpy="0 0 0"/>
     <parent link="base_link"/>
     <child link="camera_right_link"/>

Commit message: remove left and right camera

File: robot/robot_description/urdf/robot_thesis.gazebo.xacro (robot description, xacro)
@@ -125,68 +125,4 @@
     </sensor>
   </gazebo>
-  <gazebo reference="camera_left_rgb_frame">
-    <sensor type="camera" name="camera_left">
-      <always_on>true</always_on>
-      <visualize>$(arg camera_visual)</visualize>
-      <camera>
-          <horizontal_fov>${60.0*3.14/180.0}</horizontal_fov>
-          <image>
-              <width>640</width>
-              <height>480</height>
-              <format>R8G8B8</format>
-          </image>
-          <clip>
-              <near>0.03</near>
-              <far>100</far>
-          </clip>
-      </camera>
-      <plugin name="camera_controller" filename="libgazebo_ros_camera.so">
-        <alwaysOn>true</alwaysOn>
-        <updateRate>30.0</updateRate>
-        <cameraName>camera_left</cameraName>
-        <frameName>camera_left_rgb_optical_frame</frameName>
-        <imageTopicName>image_raw</imageTopicName>
-        <cameraInfoTopicName>camera_info</cameraInfoTopicName>
-        <hackBaseline>0.07</hackBaseline>
-        <distortionK1>0.0</distortionK1>
-        <distortionK2>0.0</distortionK2>
-        <distortionK3>0.0</distortionK3>
-        <distortionT1>0.0</distortionT1>
-        <distortionT2>0.0</distortionT2>
-      </plugin>
-    </sensor>
-  </gazebo>
-    <gazebo reference="camera_right_rgb_frame">
-    <sensor type="camera" name="camera_right">
-      <always_on>true</always_on>
-      <visualize>$(arg camera_visual)</visualize>
-      <camera>
-          <horizontal_fov>${60.0*3.14/180.0}</horizontal_fov>
-          <image>
-              <width>640</width>
-              <height>480</height>
-              <format>R8G8B8</format>
-          </image>
-          <clip>
-              <near>0.03</near>
-              <far>100</far>
-          </clip>
-      </camera>
-      <plugin name="camera_controller" filename="libgazebo_ros_camera.so">
-        <alwaysOn>true</alwaysOn>
-        <updateRate>30.0</updateRate>
-        <cameraName>camera_right</cameraName>
-        <frameName>camera_right_rgb_optical_frame</frameName>
-        <imageTopicName>image_raw</imageTopicName>
-        <cameraInfoTopicName>camera_info</cameraInfoTopicName>
-        <hackBaseline>0.07</hackBaseline>
-        <distortionK1>0.0</distortionK1>
-        <distortionK2>0.0</distortionK2>
-        <distortionK3>0.0</distortionK3>
-        <distortionT1>0.0</distortionT1>
-        <distortionT2>0.0</distortionT2>
-      </plugin>
-    </sensor>
-  </gazebo>
   <gazebo reference="camera_link">
       <sensor type="depth" name="camera">

File: robot/robot_description/urdf/robot_thesis.urdf.xacro (robot description, xacro)
@@ -165,54 +165,4 @@
     </inertial>
   </link>
-  <joint name="camera_left_joint" type="fixed">
-    <origin xyz="0.1 0.015 0.12" rpy="0 0 0"/>
-    <parent link="base_link"/>
-    <child link="camera_left_link"/>
-  </joint>
-  <link name="camera_left_link">
-    <collision>
-      <origin xyz="0.005 0.02 0.013" rpy="0 0 0"/>
-      <geometry>
-        <box size="0.015 0.030 0.027"/>
-      </geometry>
-    </collision>
-  </link>
-  <joint name="camera_left_rgb_joint" type="fixed">
-    <origin xyz="0.003 0.02 0.009" rpy="0 0 0"/>
-    <parent link="camera_left_link"/>
-    <child link="camera_left_rgb_frame"/>
-  </joint>
-  <link name="camera_left_rgb_frame"/>
-  <joint name="camera_left_rgb_optical_joint" type="fixed">
-    <origin xyz="0 0 0" rpy="-1.57 0 -1.57"/>
-    <parent link="camera_left_rgb_frame"/>
-    <child link="camera_left_rgb_optical_frame"/>
-  </joint>
-  <link name="camera_left_rgb_optical_frame"/>
-  <joint name="camera_right_joint" type="fixed">
-    <origin xyz="0.1 -0.015 0.12" rpy="0 0 0"/>
-    <parent link="base_link"/>
-    <child link="camera_right_link"/>
-  </joint>
-  <link name="camera_right_link">
-    <collision>
-      <origin xyz="0.005 -0.02 0.013" rpy="0 0 0"/>
-      <geometry>
-        <box size="0.015 0.030 0.027"/>
-      </geometry>
-    </collision>
-  </link>
-  <joint name="camera_right_rgb_joint" type="fixed">
-    <origin xyz="0.003 -0.02 0.009" rpy="0 0 0"/>
-    <parent link="camera_right_link"/>
-    <child link="camera_right_rgb_frame"/>
-  </joint>
-  <link name="camera_right_rgb_frame"/>
-  <joint name="camera_right_rgb_optical_joint" type="fixed">
-    <origin xyz="0 0 0" rpy="-1.57 0 -1.57"/>
-    <parent link="camera_right_rgb_frame"/>
-    <child link="camera_right_rgb_optical_frame"/>
-  </joint>
-  <link name="camera_right_rgb_optical_frame"/>
   <joint name="camera_joint" type="fixed">
     <origin xyz="0.064 -0.065 0.094" rpy="0 0 0"/>
