Commit message: add caster front link

File: robot/robot_description/urdf/robot_thesis.urdf.xacro (robot description, xacro)
@@ -105,4 +105,24 @@
   </joint>
   <link name="caster_back_link">
+    <collision>
+      <origin xyz="0 0.001 0" rpy="0 0 0"/>
+      <geometry>
+        <box size="0.030 0.009 0.020"/>
+      </geometry>
+    </collision>
+    <inertial>
+      <origin xyz="0 0 0" />
+      <mass value="0.005" />
+      <inertia ixx="0.001" ixy="0.0" ixz="0.0"
+               iyy="0.001" iyz="0.0"
+               izz="0.001" />
+    </inertial>
+  </link>
+  <joint name="caster_front_joint" type="fixed">
+    <parent link="base_link"/>
+    <child link="caster_front_link"/>
+    <origin xyz="0.081 0 -0.0025" rpy="-1.57 0 0"/>
+  </joint>
+  <link name="caster_front_link">
     <collision>
       <origin xyz="0 0.001 0" rpy="0 0 0"/>

Commit message: change robot urdf frame description

File: robot/robot_description/urdf/robot_thesis.urdf.xacro (robot description, xacro)
@@ -19,9 +19,9 @@
     <parent link="base_footprint"/>
     <child link="base_link"/>
-    <origin xyz="0.0 0.0 0.010" rpy="0 0 0"/>
+    <origin xyz="0 0 0.010" rpy="0 0 0"/>
   </joint>
   <link name="base_link">
     <visual>
-      <origin xyz="-0.0 0 0.0525" rpy="0 0 -1.5707"/>
+      <origin xyz="0 0 0.0525" rpy="0 0 -1.5707"/>
       <geometry>
         <mesh filename="package://robot_description/meshes/stl/robot_base.stl" scale="0.001 0.001 0.001"/>
@@ -30,5 +30,5 @@
     </visual>
     <collision>
-      <origin xyz="-0.0 0 0.11" rpy="0 0 0"/>
+      <origin xyz="0 0 0.11" rpy="0 0 0"/>
       <geometry>
         <cylinder length="0.11" radius="0.1"/>
@@ -151,11 +151,4 @@
   </joint>
   <link name="base_scan">
-    <!-- <visual>
-      <origin xyz="0 0 0.0" rpy="0 0 0"/>
-      <geometry>
-        <mesh filename="package://robot_description/meshes/stl/robot_lidar.stl" scale="0.001 0.001 0.001"/>
-      </geometry>
-      <material name="dark"/>
-    </visual> -->
     <collision>
       <origin xyz="0.0 0 0.05" rpy="0 0 0"/>
@@ -173,5 +166,5 @@
   </link>
   <joint name="camera_left_joint" type="fixed">
-    <origin xyz="0.1 -0.02 0.12" rpy="0 0 0"/>
+    <origin xyz="0.1 0.02 0.12" rpy="0 0 0"/>
     <parent link="base_link"/>
     <child link="camera_left_link"/>
@@ -179,5 +172,5 @@
   <link name="camera_left_link">
     <collision>
-      <origin xyz="0.005 -0.02 0.013" rpy="0 0 0"/>
+      <origin xyz="0.005 0.02 0.013" rpy="0 0 0"/>
       <geometry>
         <box size="0.015 0.030 0.027"/>
@@ -197,6 +190,6 @@
   </joint>
   <link name="camera_left_rgb_optical_frame"/>
-    <joint name="camera_right_joint" type="fixed">
-    <origin xyz="0.1 0.02 0.12" rpy="0 0 0"/>
+  <joint name="camera_right_joint" type="fixed">
+    <origin xyz="0.1 -0.02 0.12" rpy="0 0 0"/>
     <parent link="base_link"/>
     <child link="camera_right_link"/>
@@ -204,5 +197,5 @@
   <link name="camera_right_link">
     <collision>
-      <origin xyz="0.005 0.02 0.013" rpy="0 0 0"/>
+      <origin xyz="0.005 -0.02 0.013" rpy="0 0 0"/>
       <geometry>
         <box size="0.015 0.030 0.027"/>
@@ -210,6 +203,6 @@
     </collision>
   </link>
-    <joint name="camera_right_rgb_joint" type="fixed">
-    <origin xyz="0.003 0.02 0.009" rpy="0 0 0"/>
+  <joint name="camera_right_rgb_joint" type="fixed">
+    <origin xyz="0.003 -0.02 0.009" rpy="0 0 0"/>
     <parent link="camera_right_link"/>
     <child link="camera_right_rgb_frame"/>
@@ -222,48 +215,27 @@
   </joint>
   <link name="camera_right_rgb_optical_frame"/>
-    <joint name="camera_rgb_joint" type="fixed">
-      <origin xyz="${cam_px} ${kinect_cam_py} ${cam_pz}" rpy="${cam_or} ${cam_op} ${cam_oy}"/>
-      <parent link="${parent}"/>
-      <child link="camera_rgb_frame" />
-    </joint>
-    <link name="camera_rgb_frame"/>
-    <joint name="camera_rgb_optical_joint" type="fixed">
-      <origin xyz="0 0 0" rpy="${-M_PI/2} 0 ${-M_PI/2}" />
-      <parent link="camera_rgb_frame" />
-      <child link="camera_rgb_optical_frame" />
-    </joint>
-    <link name="camera_rgb_optical_frame"/>
-    <joint name="camera_joint" type="fixed">
-      <origin xyz="-0.031 ${-kinect_cam_py} -0.016" rpy="0 0 0"/>
-      <parent link="camera_rgb_frame"/>
-      <child link="camera_link"/>
-    </joint>
-      <link name="camera_link">
-<!--       <visual>
-       <origin xyz="0 0 0" rpy="0 0 ${M_PI/2}"/>
-        <geometry>
-         <mesh filename="package://turtlebot_description/meshes/sensors/kinect.dae"/>
-        </geometry>
-      </visual> -->
-      <collision>
-        <origin xyz="0.0 0.0 0.0" rpy="0 0 0"/>
-        <geometry>
-          <box size="0.07271 0.27794 0.073"/>
-        </geometry>
-      </collision>
-    </link>
-    <!-- The fixed joints & links below are usually published by static_transformers launched by the OpenNi launch
-         files. However, for Gazebo simulation we need them, so we add them here.
-         (Hence, don't publish them additionally!) -->
+  <joint name="camera_joint" type="fixed">
+    <origin xyz="0.064 -0.065 0.094" rpy="0 0 0"/>
+    <parent link="base_link"/>
+    <child link="camera_link"/>
+  </joint>
+  <link name="camera_link">
+    <collision>
+      <origin xyz="0.003 0.065 0.007" rpy="0 0 0"/>
+      <geometry>
+        <box size="0.012 0.132 0.020"/>
+      </geometry>
+    </collision>
+  </link>
   <joint name="camera_depth_joint" type="fixed">
-    <origin xyz="0 ${2 * -kinect_cam_py} 0" rpy="0 0 0" />
-    <parent link="camera_rgb_frame" />
-    <child link="camera_depth_frame" />
+    <origin xyz="${r200_cam_rgb_px} ${r200_cam_rgb_py + r200_cam_depth_offset} ${r200_cam_rgb_pz}" rpy="0 0 0"/>
+    <parent link="camera_link"/>
+    <child link="camera_depth_frame"/>
   </joint>
   <link name="camera_depth_frame"/>
   <joint name="camera_depth_optical_joint" type="fixed">
-    <origin xyz="0 0 0" rpy="${-M_PI/2} 0 ${-M_PI/2}" />
-    <parent link="camera_depth_frame" />
-    <child link="camera_depth_optical_frame" />
+    <origin xyz="0 0 0" rpy="-1.57 0 -1.57"/>
+    <parent link="camera_depth_frame"/>
+    <child link="camera_depth_optical_frame"/>
   </joint>
   <link name="camera_depth_optical_frame"/>

Commit message: update new robot visual

File: robot/robot_description/urdf/robot_thesis.urdf.xacro (robot description, xacro)
@@ -25,5 +25,5 @@
       <origin xyz="0 0 0.0525" rpy="0 0 -1.5707"/>
       <geometry>
-        <mesh filename="package://robot_description/meshes/stl/robot_base.stl" scale="0.001 0.001 0.001"/>
+        <mesh filename="package://robot_description/meshes/dae/robot_base.dae"/>
       </geometry>
       <material name="light_black"/>
@@ -51,7 +51,7 @@
   <link name="wheel_left_link">
     <visual>
-      <origin xyz="0 0 0" rpy="-1.57 0  3.14"/>
-      <geometry>
-        <mesh filename="package://robot_description/meshes/stl/robot_wheel.stl" scale="0.001 0.001 0.001"/>
+      <origin xyz="0 0 0.014" rpy="0 1.5707 0"/>
+      <geometry>
+        <mesh filename="package://robot_description/meshes/dae/robot_wheel.dae"/>
       </geometry>
       <material name="dark"/>
@@ -79,7 +79,7 @@
   <link name="wheel_right_link">
     <visual>
-      <origin xyz="0 0 0" rpy="1.57 0 0"/>
-      <geometry>
-        <mesh filename="package://robot_description/meshes/stl/robot_wheel.stl" scale="0.001 0.001 0.001"/>
+      <origin xyz="0 0 -0.014" rpy="0 -1.5707 0"/>
+      <geometry>
+        <mesh filename="package://robot_description/meshes/dae/robot_wheel.dae"/>
       </geometry>
       <material name="dark"/>

Commit message: update lidar and depth camera position

File: robot/robot_description/urdf/robot_thesis.urdf.xacro (robot description, xacro)
@@ -3,16 +3,4 @@
   <xacro:include filename="$(find robot_description)/urdf/common_properties.xacro"/>
   <xacro:include filename="$(find robot_description)/urdf/robot_thesis.gazebo.xacro"/>
-  <xacro:property name="r200_cam_rgb_px" value="0.005"/>
-  <xacro:property name="r200_cam_rgb_py" value="0.018"/>
-  <xacro:property name="r200_cam_rgb_pz" value="0.013"/>
-  <xacro:property name="r200_cam_depth_offset" value="0.01"/>
-  <xacro:property name="parent" value="base_link"/>
-  <xacro:property name="M_PI" value="3.14"/>
-  <xacro:property name="kinect_cam_py" value="-0.0125"/>
-  <xacro:property name="cam_px" value="-0.087" />
-  <xacro:property name="cam_pz" value="0.2870" />
-  <xacro:property name="cam_or" value="0" />
-  <xacro:property name="cam_op" value="0" />
-  <xacro:property name="cam_oy" value="0" />
   <link name="base_footprint"/>
   <joint name="base_joint" type="fixed">
@@ -30,7 +18,7 @@
     </visual>
     <collision>
-      <origin xyz="0 0 0.11" rpy="0 0 0"/>
+      <origin xyz="0 0 0.095" rpy="0 0 0"/>
       <geometry>
-        <cylinder length="0.11" radius="0.1"/>
+        <cylinder length="0.09" radius="0.1"/>
       </geometry>
     </collision>
@@ -148,9 +136,9 @@
     <parent link="base_link"/>
     <child link="base_scan"/>
-    <origin xyz="0.0 0 0.172" rpy="0 0 0"/>
+    <origin xyz="-0.02 0 0.172" rpy="0 0 0"/>
   </joint>
   <link name="base_scan">
     <collision>
-      <origin xyz="0.0 0 0.05" rpy="0 0 0"/>
+      <origin xyz="0.0 0 0.02" rpy="0 0 0"/>
       <geometry>
         <cylinder length="0.0315" radius="0.035"/>
@@ -166,5 +154,5 @@
   </link>
   <joint name="camera_joint" type="fixed">
-    <origin xyz="0.064 -0.065 0.094" rpy="0 0 0"/>
+    <origin xyz="0.064 -0.065 0.16" rpy="0 0 0"/>
     <parent link="base_link"/>
     <child link="camera_link"/>
@@ -174,10 +162,10 @@
       <origin xyz="0.003 0.065 0.007" rpy="0 0 0"/>
       <geometry>
-        <box size="0.012 0.132 0.020"/>
+        <box size="0.012 0.115 0.020"/>
       </geometry>
     </collision>
   </link>
   <joint name="camera_depth_joint" type="fixed">
-    <origin xyz="${r200_cam_rgb_px} ${r200_cam_rgb_py + r200_cam_depth_offset} ${r200_cam_rgb_pz}" rpy="0 0 0"/>
+    <origin xyz="0.005 0.019 0.013" rpy="0 0 0"/>
     <parent link="camera_link"/>
     <child link="camera_depth_frame"/>
