Commit message: update robot PIFBOT description

File: robot/robot_description/urdf/PIFBOT/robot_PIFBOT.gazebo.xacro (robot description, xacro)
@@ -1,4 +1,4 @@
 <?xml version="1.0"?>
-<robot name="robot_thesis_sim" xmlns:xacro="http://ros.org/wiki/xacro">
+<robot name="robot_PIFBOT_sim" xmlns:xacro="http://ros.org/wiki/xacro">
   <xacro:arg name="laser_visual" default="false"/>
   <xacro:arg name="imu_visual"   default="false"/>

File: robot/robot_description/urdf/PIFBOT/robot_PIFBOT.urdf.xacro (robot description, xacro)
@@ -1,6 +1,6 @@
 <?xml version="1.0" ?>
-<robot name="robot_thesis" xmlns:xacro="http://ros.org/wiki/xacro">
+<robot name="robot_PIFBOT" xmlns:xacro="http://ros.org/wiki/xacro">
   <xacro:include filename="$(find robot_description)/urdf/common_properties.xacro"/>
-  <xacro:include filename="$(find robot_description)/urdf/robot_thesis.gazebo.xacro"/>
+  <xacro:include filename="$(find robot_description)/urdf/PIFBOT/robot_PIFBOT.gazebo.xacro"/>
   <link name="base_footprint"/>
   <joint name="base_joint" type="fixed">
@@ -13,5 +13,5 @@
       <origin xyz="0 0 0.0525" rpy="0 0 -1.5707"/>
       <geometry>
-        <mesh filename="package://robot_description/meshes/dae/robot_base.dae"/>
+        <mesh filename="package://robot_description/meshes/PIFBOT/dae/robot_base.dae"/>
       </geometry>
       <material name="light_black"/>
@@ -41,5 +41,5 @@
       <origin xyz="0 0 0.014" rpy="0 1.5707 0"/>
       <geometry>
-        <mesh filename="package://robot_description/meshes/dae/robot_wheel.dae"/>
+        <mesh filename="package://robot_description/meshes/PIFBOT/dae/robot_wheel.dae"/>
       </geometry>
       <material name="dark"/>
@@ -69,5 +69,5 @@
       <origin xyz="0 0 -0.014" rpy="0 -1.5707 0"/>
       <geometry>
-        <mesh filename="package://robot_description/meshes/dae/robot_wheel.dae"/>
+        <mesh filename="package://robot_description/meshes/PIFBOT/dae/robot_wheel.dae"/>
       </geometry>
       <material name="dark"/>
